Commit message: Done with 25 (part I)

File: body.urdf (robot description, URDF)
Before this commit: robot robot, 0 links, 0 joints
Links:
- added link BackLeg, mass 1; collision box size=1 1 1; visual box size=1 1 1
- added link FrontLeg, mass 1; collision box size=1 1 1; visual box size=1 1 1
- added link Torso, mass 1; collision box size=1 1 1; visual box size=1 1 1
Joints:
- added joint Torso_BackLeg: type revolute, parent Torso, child BackLeg, origin xyz=1 0 1 rpy=0 0 0, axis 0 1 0, limit lower=-3.14159 upper=3.14159 effort=0.0 velocity=0.0
- added joint Torso_FrontLeg: type revolute, parent Torso, child FrontLeg, origin xyz=2 0 1 rpy=0 0 0, axis 0 1 0, limit lower=-3.14159 upper=3.14159 effort=0.0 velocity=0.0

Commit message: 45 Biasing Evolution (N)

File: body.urdf (robot description, URDF)
Before this commit: robot robot, 3 links, 2 joints
Links:
- added link LeftLeg, mass 1; collision box size=1 0.2 0.2; visual box size=1 0.2 0.2
- added link LowerBackLeg, mass 1; collision box size=0.2 0.2 1; visual box size=0.2 0.2 1
- added link LowerFrontLeg, mass 1; collision box size=0.2 0.2 1; visual box size=0.2 0.2 1
- added link LowerLeftLeg, mass 1; collision box size=0.2 0.2 1; visual box size=0.2 0.2 1
- added link LowerRightLeg, mass 1; collision box size=0.2 0.2 1; visual box size=0.2 0.2 1
- added link RightLeg, mass 1; collision box size=1 0.2 0.2; visual box size=1 0.2 0.2
Joints:
- added joint BackLeg_LowerBackLeg: type revolute, parent BackLeg, child LowerBackLeg, origin xyz=0 -1 0 rpy=0 0 0, axis 1 0 0, limit lower=-3.14159 upper=3.14159 effort=0.0 velocity=0.0
- added joint FrontLeg_LowerFrontLeg: type revolute, parent FrontLeg, child LowerFrontLeg, origin xyz=0 1 0 rpy=0 0 0, axis 1 0 0, limit lower=-3.14159 upper=3.14159 effort=0.0 velocity=0.0
- added joint LeftLeg_LowerLeftLeg: type revolute, parent LeftLeg, child LowerLeftLeg, origin xyz=-1 0 0 rpy=0 0 0, axis 0 1 0, limit lower=-3.14159 upper=3.14159 effort=0.0 velocity=0.0
- added joint RightLeg_LowerRightLeg: type revolute, parent RightLeg, child LowerRightLeg, origin xyz=1 0 0 rpy=0 0 0, axis 0 1 0, limit lower=-3.14159 upper=3.14159 effort=0.0 velocity=0.0
- added joint Torso_LeftLeg: type revolute, parent Torso, child LeftLeg, origin xyz=-0.5 0 1 rpy=0 0 0, axis 0 1 0, limit lower=-3.14159 upper=3.14159 effort=0.0 velocity=0.0
- added joint Torso_RightLeg: type revolute, parent Torso, child RightLeg, origin xyz=0.5 0 1 rpy=0 0 0, axis 0 1 0, limit lower=-3.14159 upper=3.14159 effort=0.0 velocity=0.0
- joint Torso_BackLeg: axis 0 1 0 -> 1 0 0
- joint Torso_FrontLeg: axis 0 1 0 -> 1 0 0

Commit message: Completed FinalProject

File: body.urdf (robot description, URDF)
Before this commit: robot robot, 9 links, 8 joints
Links:
- removed link LowerBackLeg
- removed link LowerFrontLeg
- removed link LowerLeftLeg
- removed link LowerRightLeg
- removed link Torso
- added link Turtle, mass 1; collision box size=2 2 0.2; visual box size=2 2 0.2
Joints:
- removed joint BackLeg_LowerBackLeg
- removed joint FrontLeg_LowerFrontLeg
- removed joint LeftLeg_LowerLeftLeg
- removed joint RightLeg_LowerRightLeg
- removed joint Torso_BackLeg
- removed joint Torso_FrontLeg
- removed joint Torso_LeftLeg
- removed joint Torso_RightLeg
- added joint Turtle_BackLeg: type revolute, parent Turtle, child BackLeg, origin xyz=0 -0.75 1 rpy=0 0 0, axis 1 0 -1, limit lower=-3.14159 upper=3.14159 effort=0.0 velocity=0.0
- added joint Turtle_FrontLeg: type revolute, parent Turtle, child FrontLeg, origin xyz=0 0.75 1 rpy=0 0 0, axis 1 0 -1, limit lower=-3.14159 upper=3.14159 effort=0.0 velocity=0.0
- added joint Turtle_LeftLeg: type revolute, parent Turtle, child LeftLeg, origin xyz=-0.75 0 1 rpy=0 0 0, axis 0 1 -1, limit lower=-3.14159 upper=3.14159 effort=0.0 velocity=0.0
- added joint Turtle_RightLeg: type revolute, parent Turtle, child RightLeg, origin xyz=0.75 0 1 rpy=0 0 0, axis 0 1 -1, limit lower=-3.14159 upper=3.14159 effort=0.0 velocity=0.0

Commit message: Snake Random

File: body.urdf (robot description, URDF)
Before this commit: robot robot, 5 links, 4 joints
Links:
- removed link BackLeg
- removed link FrontLeg
- removed link LeftLeg
- removed link RightLeg
- removed link Turtle
- added link Head, mass 1; collision box size=1 4 1; visual box size=1 4 1
- added link Link0, mass 1; collision box size=2 4 1; visual box size=2 4 1
- added link Link1, mass 1; collision box size=3 4 3; visual box size=3 4 3
- added link Link2, mass 1; collision box size=3 4 2; visual box size=3 4 2
- added link Link3, mass 1; collision box size=2 4 1; visual box size=2 4 1
- added link Link4, mass 1; collision box size=2 4 1; visual box size=2 4 1
- added link Link5, mass 1; collision box size=2 4 2; visual box size=2 4 2
- added link Link6, mass 1; collision box size=2 4 3; visual box size=2 4 3
- added link Link7, mass 1; collision box size=2 4 1; visual box size=2 4 1
Joints:
- removed joint Turtle_BackLeg
- removed joint Turtle_FrontLeg
- removed joint Turtle_LeftLeg
- removed joint Turtle_RightLeg
- added joint Head_Link0: type revolute, parent Head, child Link0, origin xyz=0 8.666666666666666 3 rpy=0 0 0, axis 0 0 1, limit lower=-3.14159 upper=3.14159 effort=0.0 velocity=0.0
- added joint Link0_Link1: type revolute, parent Link0, child Link1, origin xyz=0 -4 0 rpy=0 0 0, axis 0 0 1, limit lower=-3.14159 upper=3.14159 effort=0.0 velocity=0.0
- added joint Link1_Link2: type revolute, parent Link1, child Link2, origin xyz=0 -4 0 rpy=0 0 0, axis 0 0 1, limit lower=-3.14159 upper=3.14159 effort=0.0 velocity=0.0
- added joint Link2_Link3: type revolute, parent Link2, child Link3, origin xyz=0 -4 0 rpy=0 0 0, axis 0 0 1, limit lower=-3.14159 upper=3.14159 effort=0.0 velocity=0.0
- added joint Link3_Link4: type revolute, parent Link3, child Link4, origin xyz=0 -4 0 rpy=0 0 0, axis 0 0 1, limit lower=-3.14159 upper=3.14159 effort=0.0 velocity=0.0
- added joint Link4_Link5: type revolute, parent Link4, child Link5, origin xyz=0 -4 0 rpy=0 0 0, axis 0 0 1, limit lower=-3.14159 upper=3.14159 effort=0.0 velocity=0.0
- added joint Link5_Link6: type revolute, parent Link5, child Link6, origin xyz=0 -4 0 rpy=0 0 0, axis 0 0 1, limit lower=-3.14159 upper=3.14159 effort=0.0 velocity=0.0
- added joint Link6_Link7: type revolute, parent Link6, child Link7, origin xyz=0 -4 0 rpy=0 0 0, axis 0 0 1, limit lower=-3.14159 upper=3.14159 effort=0.0 velocity=0.0

Commit message: bugfix

File: body.urdf (robot description, URDF)
Before this commit: robot robot, 9 links, 8 joints
Links:
- added link Link8, mass 1; collision box size=1 2 3; visual box size=1 2 3
- link Head: geometry collision box size=3 2 3; visual box size=3 2 3
- link Link0: geometry collision box size=3 2 1; visual box size=3 2 1
- link Link1: geometry collision box size=1 2 3; visual box size=1 2 3
- link Link2: geometry collision box size=3 2 1; visual box size=3 2 1
- link Link3: geometry collision box size=1 2 3; visual box size=1 2 3
- link Link4: geometry collision box size=2 2 3; visual box size=2 2 3
- link Link5: geometry collision box size=3 2 1; visual box size=3 2 1
- link Link6: geometry collision box size=1 2 1; visual box size=1 2 1
- link Link7: geometry collision box size=2 2 1; visual box size=2 2 1
Joints:
- added joint Link7_Link8: type revolute, parent Link7, child Link8, origin xyz=0 -2 0 rpy=0 0 0, axis 0 0 1, limit lower=-3.14159 upper=3.14159 effort=0.0 velocity=0.0
- joint Head_Link0: origin xyz=0 8.666666666666666 3 rpy=0 0 0 -> xyz=0 9.333333333333334 3 rpy=0 0 0
- joint Link0_Link1: origin xyz=0 -4 0 rpy=0 0 0 -> xyz=0 -2 0 rpy=0 0 0
- joint Link1_Link2: origin xyz=0 -4 0 rpy=0 0 0 -> xyz=0 -2 0 rpy=0 0 0
- joint Link2_Link3: origin xyz=0 -4 0 rpy=0 0 0 -> xyz=0 -2 0 rpy=0 0 0
- joint Link3_Link4: origin xyz=0 -4 0 rpy=0 0 0 -> xyz=0 -2 0 rpy=0 0 0
- joint Link4_Link5: origin xyz=0 -4 0 rpy=0 0 0 -> xyz=0 -2 0 rpy=0 0 0
- joint Link5_Link6: origin xyz=0 -4 0 rpy=0 0 0 -> xyz=0 -2 0 rpy=0 0 0
- joint Link6_Link7: origin xyz=0 -4 0 rpy=0 0 0 -> xyz=0 -2 0 rpy=0 0 0

Commit message: s

File: body.urdf (robot description, URDF)
Before this commit: robot robot, 10 links, 9 joints
Links:
- removed link Link5
- removed link Link6
- removed link Link7
- removed link Link8
- link Head: geometry collision box size=2 4 1; visual box size=2 4 1
- link Link0: geometry collision box size=1 4 2; visual box size=1 4 2
- link Link1: geometry collision box size=2 4 3; visual box size=2 4 3
- link Link2: geometry collision box size=1 4 1; visual box size=1 4 1
- link Link3: geometry collision box size=1 4 1; visual box size=1 4 1
- link Link4: geometry collision box size=1 4 3; visual box size=1 4 3
Joints:
- removed joint Link4_Link5
- removed joint Link5_Link6
- removed joint Link6_Link7
- removed joint Link7_Link8
- joint Head_Link0: origin xyz=0 9.333333333333334 3 rpy=0 0 0 -> xyz=0 8.666666666666666 3 rpy=0 0 0
- joint Link0_Link1: origin xyz=0 -2 0 rpy=0 0 0 -> xyz=0 -4 0 rpy=0 0 0
- joint Link1_Link2: origin xyz=0 -2 0 rpy=0 0 0 -> xyz=0 -4 0 rpy=0 0 0
- joint Link2_Link3: origin xyz=0 -2 0 rpy=0 0 0 -> xyz=0 -4 0 rpy=0 0 0
- joint Link3_Link4: origin xyz=0 -2 0 rpy=0 0 0 -> xyz=0 -4 0 rpy=0 0 0

Commit message: Assignment 7

File: body.urdf (robot description, URDF)
Before this commit: robot robot, 6 links, 5 joints
Links:
- removed link Head
- removed link Link4
- link Link0: geometry collision box size=0.9754370689594419 0.6782674854632328 0.6782674854632328; visual box size=0.9754370689594419 0.6782674854632328 0.6782674854632328
- link Link1: geometry collision box size=0.576726471736457 0.5731587660224584 0.5731587660224584; visual box size=0.576726471736457 0.5731587660224584 0.5731587660224584
- link Link2: geometry collision box size=0.8117559559684958 0.14561936621141713 0.14561936621141713; visual box size=0.8117559559684958 0.14561936621141713 0.14561936621141713
- link Link3: geometry collision box size=0.9528238634118608 0.20869182253695784 0.20869182253695784; visual box size=0.9528238634118608 0.20869182253695784 0.20869182253695784
Joints:
- removed joint Head_Link0
- removed joint Link3_Link4
- joint Link0_Link1: axis 0 0 1 -> 0.2669608002245988 0.21233147286200105 0.13191978404122884; origin xyz=0 -4 0 rpy=0 0 0 -> xyz=-0.48771853447972097 -0.3391337427316164 0 rpy=0 0 0
- joint Link1_Link2: axis 0 0 1 -> 0.861680518685561 0.4745663041875784 0.34774729539941196; origin xyz=0 -4 0 rpy=0 0 0 -> xyz=-0.2883632358682285 0 0 rpy=0 0 0
- joint Link2_Link3: axis 0 0 1 -> 0.2885965424238903 0.22710678912982896 0.1718536232085759; origin xyz=0 -4 0 rpy=0 0 0 -> xyz=0 0 0 rpy=0 0 0

Commit message: Assignment8

File: body.urdf (robot description, URDF)
Before this commit: robot robot, 4 links, 3 joints
Links:
- link Link0: geometry collision box size=0.8268495298164329 0.4710309799729654 0.4710309799729654; visual box size=0.8268495298164329 0.4710309799729654 0.4710309799729654
- link Link1: geometry collision box size=0.20905258484906086 0.4922610991810721 0.4922610991810721; visual box size=0.20905258484906086 0.4922610991810721 0.4922610991810721
- link Link2: geometry collision box size=0.2919569015898764 0.951055271479538 0.951055271479538; visual box size=0.2919569015898764 0.951055271479538 0.951055271479538
- link Link3: geometry collision box size=0.8074398138807576 0.1768955740321151 0.1768955740321151; visual box size=0.8074398138807576 0.1768955740321151 0.1768955740321151
Joints:
- joint Link0_Link1: axis 0.2669608002245988 0.21233147286200105 0.13191978404122884 -> 0.8121281847341797 0.8083701151567984 0.8312786859905937; origin xyz=-0.48771853447972097 -0.3391337427316164 0 rpy=0 0 0 -> xyz=0.41342476490821645 0 0.2355154899864827 rpy=0 0 0
- joint Link1_Link2: axis 0.861680518685561 0.4745663041875784 0.34774729539941196 -> 0.7760336969528621 0.21468845490656652 0.9080948769971683; origin xyz=-0.2883632358682285 0 0 rpy=0 0 0 -> xyz=-0.10452629242453043 0 0 rpy=0 0 0
- joint Link2_Link3: axis 0.2885965424238903 0.22710678912982896 0.1718536232085759 -> 0.5829138293521593 0.9455934128787277 0.6926426689019555; origin xyz=0 0 0 rpy=0 0 0 -> xyz=0.1459784507949382 0 0 rpy=0 0 0

Commit message: Revert "Assignment8"
This reverts commit 101083a1ddb128bf1d476e340c21310e7e5dfce9.

File: body.urdf (robot description, URDF)
Before this commit: robot robot, 4 links, 3 joints
Links:
- link Link0: geometry collision box size=0.9754370689594419 0.6782674854632328 0.6782674854632328; visual box size=0.9754370689594419 0.6782674854632328 0.6782674854632328
- link Link1: geometry collision box size=0.576726471736457 0.5731587660224584 0.5731587660224584; visual box size=0.576726471736457 0.5731587660224584 0.5731587660224584
- link Link2: geometry collision box size=0.8117559559684958 0.14561936621141713 0.14561936621141713; visual box size=0.8117559559684958 0.14561936621141713 0.14561936621141713
- link Link3: geometry collision box size=0.9528238634118608 0.20869182253695784 0.20869182253695784; visual box size=0.9528238634118608 0.20869182253695784 0.20869182253695784
Joints:
- joint Link0_Link1: axis 0.8121281847341797 0.8083701151567984 0.8312786859905937 -> 0.2669608002245988 0.21233147286200105 0.13191978404122884; origin xyz=0.41342476490821645 0 0.2355154899864827 rpy=0 0 0 -> xyz=-0.48771853447972097 -0.3391337427316164 0 rpy=0 0 0
- joint Link1_Link2: axis 0.7760336969528621 0.21468845490656652 0.9080948769971683 -> 0.861680518685561 0.4745663041875784 0.34774729539941196; origin xyz=-0.10452629242453043 0 0 rpy=0 0 0 -> xyz=-0.2883632358682285 0 0 rpy=0 0 0
- joint Link2_Link3: axis 0.5829138293521593 0.9455934128787277 0.6926426689019555 -> 0.2885965424238903 0.22710678912982896 0.1718536232085759; origin xyz=0.1459784507949382 0 0 rpy=0 0 0 -> xyz=0 0 0 rpy=0 0 0
